Commit message: Rebase from 'upstream'

File: cpr_agriculture_gazebo/urdf/agriculture_geometry.urdf.xacro (robot description, xacro)
@@ -7,6 +7,9 @@
       <inertia ixx="1" ixy="0" ixz="0" iyy="1" iyz="0" izz="1"/>
     </inertial>
+    <!--
+      Align the world geometry so that X+ is east and Y+ is north (ENU)
+    -->
     <visual>
-      <origin xyz="0 0 0" rpy="0 0 0"/>
+      <origin xyz="0 0 0" rpy="0 0 ${pi}"/>
       <geometry>
         <mesh filename="package://cpr_agriculture_gazebo/meshes/agriculture_world.dae"/>
@@ -14,5 +17,5 @@
     </visual>
     <collision>
-      <origin xyz="0 0 0" rpy="0 0 0"/>
+      <origin xyz="0 0 0" rpy="0 0 ${pi}"/>
       <geometry>
         <mesh filename="package://cpr_agriculture_gazebo/meshes/agriculture_world.dae"/>
@@ -28,4 +31,12 @@
     </collision>
   </link>
+  <xacro:include filename="$(find cpr_accessories_gazebo)/urdf/base_station.urdf.xacro" />
+  <xacro:cpr_base_station name="base_station" parent="agriculture_world_link">
+    <origin xyz="-17 40 0.7" />
+  </xacro:cpr_base_station>
+  <xacro:include  filename="$(find cpr_accessories_gazebo)/urdf/charge_dock.urdf.xacro" />
+  <xacro:cpr_charge_dock name="charge_dock" parent="agriculture_world_link">
+    <origin xyz="8 -4 -0.2" rpy="0 0 1.5707963267948966" />
+  </xacro:cpr_charge_dock>
   <gazebo> <static>true</static></gazebo>
 </robot>

File: cpr_inspection_gazebo/urdf/inspection_geometry.urdf.xacro (robot description, xacro)
@@ -8,19 +8,19 @@
     </inertial>
     <visual>
-      <origin xyz="0 0 0" rpy="0 0 0"/>
+      <origin xyz="0 0 0" rpy="0 0 3.141592653589793"/>
       <geometry>
-        <mesh filename="package://cpr_inspection_gazebo/meshes/inspection_world.dae"/>
+        <mesh filename="package://cpr_inspection_gazebo/meshes/inspection_world.dae" scale="2 2 1"/>
       </geometry>
     </visual>
     <visual>
-      <origin xyz="0 0 0" rpy="0 0 0"/>
+      <origin xyz="0 0 0" rpy="0 0 3.141592653589793"/>
       <geometry>
-        <mesh filename="package://cpr_inspection_gazebo/meshes/inspection_water.dae"/>
+        <mesh filename="package://cpr_inspection_gazebo/meshes/inspection_water.dae" scale="2 2 1"/>
       </geometry>
     </visual>
     <collision>
-      <origin xyz="0 0 0" rpy="0 0 0"/>
+      <origin xyz="0 0 0" rpy="0 0 3.141592653589793"/>
       <geometry>
-        <mesh filename="package://cpr_inspection_gazebo/meshes/inspection_world.dae"/>
+        <mesh filename="package://cpr_inspection_gazebo/meshes/inspection_world.dae" scale="2 2 1"/>
       </geometry>
       <surface>
@@ -34,4 +34,8 @@
     </collision>
   </link>
+  <xacro:include filename="$(find cpr_accessories_gazebo)/urdf/base_station.urdf.xacro" />
+  <xacro:cpr_base_station name="base_station" parent="inspection_world_link">
+    <origin xyz="0 -12 1" rpy="0 0 0" />
+  </xacro:cpr_base_station>
   <gazebo> <static>true</static></gazebo>
 </robot>

File: cpr_orchard_gazebo/urdf/orchard_geometry.urdf.xacro (robot description, xacro)
@@ -8,5 +8,5 @@
     </inertial>
     <visual>
-      <origin xyz="0 0 0" rpy="0 0 0"/>
+      <origin xyz="0 0 0" rpy="0 0 1.5707963267948966"/>
       <geometry>
         <mesh filename="package://cpr_orchard_gazebo/meshes/orchard_world.dae"/>
@@ -14,5 +14,5 @@
     </visual>
     <visual>
-      <origin xyz="0 0 0" rpy="0 0 0"/>
+      <origin xyz="0 0 0" rpy="0 0 1.5707963267948966"/>
       <geometry>
         <mesh filename="package://cpr_orchard_gazebo/meshes/orchard_trunks.dae"/>
@@ -20,5 +20,5 @@
     </visual>
     <visual>
-      <origin xyz="0 0 0" rpy="0 0 0"/>
+      <origin xyz="0 0 0" rpy="0 0 1.5707963267948966"/>
       <geometry>
         <mesh filename="package://cpr_orchard_gazebo/meshes/orchard_leaves.dae"/>
@@ -26,5 +26,5 @@
     </visual>
     <collision>
-      <origin xyz="0 0 0" rpy="0 0 0"/>
+      <origin xyz="0 0 0" rpy="0 0 1.5707963267948966"/>
       <geometry>
         <mesh filename="package://cpr_orchard_gazebo/meshes/orchard_world.dae"/>
@@ -40,5 +40,5 @@
     </collision>
     <collision>
-      <origin xyz="0 0 0" rpy="0 0 0"/>
+      <origin xyz="0 0 0" rpy="0 0 1.5707963267948966"/>
       <geometry>
         <mesh filename="package://cpr_orchard_gazebo/meshes/orchard_trunks.dae"/>
@@ -47,3 +47,7 @@
   </link>
   <gazebo> <static>true</static></gazebo>
+  <xacro:include filename="$(find cpr_accessories_gazebo)/urdf/base_station.urdf.xacro" />
+  <xacro:cpr_base_station name="base_station" parent="orchard_world_link">
+    <origin xyz="-2 1 0" />
+  </xacro:cpr_base_station>
 </robot>
